Commit message: add i3dr camera urdf generator

File: urdf/i3dr_stereo_camera.urdf.xacro (robot description, xacro)
@@ -4,49 +4,54 @@
 -->
 <robot xmlns:xacro="http://ros.org/wiki/xacro">
-    <xacro:macro name="i3dr_stereo_camera">
+    <xacro:macro name="i3dr_stereo_camera" params="camera_name baseline toe_in width height length image_format:=RGB8 image_height:=640 image_width:=480 hfov:=1.579 focus_near:=0 focus_far:=100 camera_offset_x:=0 camera_offset_y:=0 camera_offset_z:=0 mount_offset_x:=0 mount_offset_y:=0 mount_offset_z:=0 r:=1 g:=0 b:=0 a:=1">
         <link name="${camera_name}_cameraLeft_optical" />
         <link name="${camera_name}_cameraRight_optical" />
         <link name="${camera_name}_cameraLeft" />
         <link name="${camera_name}_cameraRight" />
+        <link name="${camera_name}_base_link" />
         <link name="${camera_name}_center">
             <visual>
                 <origin xyz="0 0 0" rpy="0 0 0"/>
                 <geometry>
-                    <box size="0.140 0.390 0.05"/>
+                    <box size="${width} ${height} ${length}"/>
                 </geometry>
-                <material name="Orange">
-                    <color rgba="1 0.5 0 1"/>
+                <material name="${camera_name}_camera_colour">
+                    <color rgba="${r} ${g} ${b} ${a}"/>
                 </material>
             </visual>
         </link>
-        <link name="${camera_name}_depth_camera" />
         <joint name="${camera_name}_right_camera_joint" type="fixed">
             <parent link="${camera_name}_center"/>
             <child link="${camera_name}_cameraRight"/>
-            <!--<origin xyz="0.0245 0.148794 0.086874" rpy="0 0 0" />-->
-            <origin xyz="0.086874 -0.148794  0.0245" rpy="0 0 0" />
+            <origin xyz="${camera_offset_x} -${(baseline/2)+camera_offset_y} ${camera_offset_z}" rpy="0 0 0" />
         </joint>
         <joint name="${camera_name}_left_camera_joint" type="fixed">
             <parent link="${camera_name}_center"/>
             <child link="${camera_name}_cameraLeft"/>
-            <!--<origin xyz="0.0245 -0.148794 0.086874" rpy="0 0 0" />-->
-            <origin xyz="0.086874 0.148794 0.0245" rpy="0 0 0" />
+            <origin xyz="${camera_offset_x} ${(baseline/2)+camera_offset_y} ${camera_offset_z}" rpy="0 0 0" />
         </joint>
         <joint name="${camera_name}_left_optical_joint" type="fixed">
             <parent link="${camera_name}_cameraLeft"/>
             <child link="${camera_name}_cameraLeft_optical"/>
-        <!-- Correct for the optical frame orientation -->
-            <origin xyz="0 0 0" rpy="${-pi/2} 0 ${-pi/2}" />
+            <!-- Correct for the optical frame orientation -->
+            <origin xyz="0 0 0" rpy="${-pi/2} 0 ${(-pi/2)-toe_in}" />
         </joint>
         <joint name="${camera_name}_right_optical_joint" type="fixed">
             <parent link="${camera_name}_cameraRight"/>
             <child link="${camera_name}_cameraRight_optical"/>
-        <!-- Correct for the optical frame orientation -->
-            <origin xyz="0 0 0" rpy="${-pi/2} 0 ${-pi/2}" />
+            <!-- Correct for the optical frame orientation -->
+            <origin xyz="0 0 0" rpy="${-pi/2} 0 ${(-pi/2)+toe_in}" />
         </joint>
-        <joint name="${camera_name}_depth_camera_joint" type="fixed">
-            <parent link="${camera_name}_cameraLeft"/>
-            <child link="${camera_name}_depth_camera"/>
-            <origin xyz="0 0 0" rpy="0 0 0" />
+        <sensor name="${camera_name}_right_camera_sensor" update_rate="60">
+            <parent link="${camera_name}_cameraRight_optical"/>
+            <origin xyz="0 0 0" rpy="0 0 0"/>
+            <camera>
+                <image width="${image_width}" height="${image_height}" hfov="${hfov}" format="${image_format}" near="${focus_near}" far="${focus_far}"/>
+            </camera>
+        </sensor>
+        <joint name="${camera_name}_mount_center_joint" type="fixed">
+            <parent link="${camera_name}_base_link"/>
+            <child link="${camera_name}_center"/>
+            <origin xyz="${mount_offset_x} ${mount_offset_y} ${(length/2)+mount_offset_z}" rpy="0 0 0" />
         </joint>
     </xacro:macro>

Commit message: Added gazebo plugins

File: urdf/i3dr_stereo_camera.urdf.xacro (robot description, xacro)
@@ -4,5 +4,11 @@
 -->
 <robot xmlns:xacro="http://ros.org/wiki/xacro">
-    <xacro:macro name="i3dr_stereo_camera" params="camera_name baseline toe_in width height length image_format:=RGB8 image_height:=640 image_width:=480 hfov:=1.579 focus_near:=0 focus_far:=100 camera_offset_x:=0 camera_offset_y:=0 camera_offset_z:=0 mount_offset_x:=0 mount_offset_y:=0 mount_offset_z:=0 r:=1 g:=0 b:=0 a:=1">
+    <xacro:macro name="i3dr_stereo_camera" params="camera_name baseline toe_in width height length
+    image_format:=RGB8
+    image_height:=640 image_width:=480
+    hfov:=1.579 focus_near:=0 focus_far:=100
+    camera_offset_x:=0 camera_offset_y:=0 camera_offset_z:=0
+    mount_offset_x:=0 mount_offset_y:=0 mount_offset_z:=0
+    r:=1 g:=0 b:=0 a:=1">
         <link name="${camera_name}_cameraLeft_optical" />
         <link name="${camera_name}_cameraRight_optical" />
@@ -55,4 +61,90 @@
             <origin xyz="${mount_offset_x} ${mount_offset_y} ${(length/2)+mount_offset_z}" rpy="0 0 0" />
         </joint>
+        <gazebo reference="${camera_name}_cameraLeft">
+          <sensor type="multicamera" name="stereo_camera">
+            <update_rate>0.5</update_rate> <!-- reality 60fps on USB3-->
+            <camera name="left">
+                <horizontal_fov>1.579</horizontal_fov>
+                <image>
+                    <width>320</width>
+                    <height>240</height>
+                    <format>L8</format>
+                </image>
+                <clip>
+                    <near>0.02</near>
+                    <far>300</far>
+                </clip>
+                <noise>
+                    <type>gaussian</type>
+                    <mean>0.0</mean>
+                    <stddev>0.007</stddev>
+                </noise>
+            </camera>
+            <camera name="right">
+                <pose>0 -0.07 0 0 0 0</pose>
+                <horizontal_fov>1.579</horizontal_fov>
+                <image>
+                    <width>320</width>
+                    <height>240</height>
+                    <format>L8</format>
+                </image>
+                <clip>
+                    <near>0.02</near>
+                    <far>300</far>
+                </clip>
+                <noise>
+                    <type>gaussian</type>
+                    <mean>0.0</mean>
+                    <stddev>0.007</stddev>
+                </noise>
+            </camera>
+            <plugin name="stereo_camera_controller" filename="libgazebo_ros_multicamera.so">
+                <alwaysOn>true</alwaysOn>
+                <updateRate>1</updateRate>
+                <cameraName>${camera_name}</cameraName>
+                <imageTopicName>image_raw</imageTopicName>
+                <cameraInfoTopicName>camera_info</cameraInfoTopicName>
+                <frameName>${camera_name}_cameraLeft_optical</frameName>
+                <hackBaseline>0.07</hackBaseline>
+                <distortionK1>0.0</distortionK1>
+                <distortionK2>0.0</distortionK2>
+                <distortionK3>0.0</distortionK3>
+                <distortionT1>0.0</distortionT1>
+                <distortionT2>0.0</distortionT2>
+            </plugin>
+          </sensor>
+        </gazebo>
+        <gazebo reference="${camera_name}_cameraLeft">
+          <sensor type="depth" name="${camera_name}_depth_camera">
+            <update_rate>1</update_rate>
+            <camera>
+              <horizontal_fov>${62.8 * pi/180.0}</horizontal_fov>
+              <image>
+                <format>R8G8B8</format>
+                <width>160</width>
+                <height>120</height>
+              </image>
+              <clip>
+                <near>0.05</near>
+                <far>12</far>
+              </clip>
+            </camera>
+            <plugin name="${camera_name}_depth_camera_controller" filename="libgazebo_ros_openni_kinect.so">
+              <alwaysOn>true</alwaysOn>
+              <updateRate>1</updateRate>
+              <imageTopicName>${camera_name}_depth/image_raw</imageTopicName>
+              <cameraInfoTopicName>${camera_name}_depth/camera_info</cameraInfoTopicName>
+              <depthImageTopicName>${camera_name}_depth/depth/image_raw</depthImageTopicName>
+              <depthImageCameraInfoTopicName>${camera_name}_depth/depth/camera_info</depthImageCameraInfoTopicName>
+              <pointCloudTopicName>${camera_name}_depth/depth/points</pointCloudTopicName>
+              <frameName>${camera_name}_cameraLeft_optical</frameName>
+              <distortion_k1>0.0</distortion_k1>
+              <distortion_k2>0.0</distortion_k2>
+              <distortion_k3>0.0</distortion_k3>
+              <distortion_t1>0.0</distortion_t1>
+              <distortion_t2>0.0</distortion_t2>
+            </plugin>
+          </sensor>
+        </gazebo>
     </xacro:macro>
 </robot>
