Commit message: Package tidy up, fix IMU timestamps, fix duplicate camera info manager, update urdf and docs

File: urdf/deimos.urdf.xacro (robot description, xacro)
@@ -15,5 +15,5 @@
             <geometry>
                 <box size="0.0324 0.101 0.038"/>
-                <!--mesh filename="package://deimos-ros/urdf/deimos.stl" /-->
+                <!--mesh filename="package://deimos/urdf/deimos.stl" /-->
             </geometry>
         </visual>
@@ -21,8 +21,16 @@
     <link name="deimos_depth_camera" />
     <link name="imu_link"/>
+    <!-- M4 trisert location -->
+    <link name="deimos_left_mount" />
+    <link name="deimos_right_mount" />
     <!-- Deimos has a 60 mm baseline -->
-    <joint name="deimos_left_camera_joint" type="fixed">
-        <parent link="deimos_center"/>
-        <child link="cameraLeft"/>
+    <joint name="deimos_left_mount_joint" type="fixed">
+        <parent link="deimos_left_mount"/>
+        <child link="deimos_center"/>
+        <origin xyz="-0.13241 -${-0.017875+0.03} 0.025" rpy="0 0 0" />
+    </joint>
+    <joint name="deimos_right_mount_joint" type="fixed">
+        <parent link="deimos_left_mount"/>
+        <child link="deimos_right_mount"/>
         <origin xyz="0 0.03 0" rpy="0 0 0" />
     </joint>
@@ -30,4 +38,9 @@
         <parent link="deimos_center"/>
         <child link="cameraRight"/>
+        <origin xyz="0 0.03 0" rpy="0 0 0" />
+    </joint>
+    <joint name="deimos_left_camera_joint" type="fixed">
+        <parent link="deimos_center"/>
+        <child link="cameraLeft"/>
         <origin xyz="0 -0.03 0" rpy="0 0 0" />
     </joint>
@@ -51,5 +64,5 @@
     <!-- Correct for IMU orientation, Z -> X -->
     <joint name="imu_joint" type="fixed">
-    	<origin xyz="0 0 0" rpy="0 ${M_PI/2} 0" />
+    	<origin xyz="0 0.015 -0.002" rpy="0 ${M_PI/2} 0" />
     	<parent link="deimos_center" />
     	<child link="imu_link" />

File: urdf/standalone.urdf.xacro (robot description, xacro)
@@ -7,5 +7,5 @@
     <origin xyz="0 0 0" rpy="0 0 0" />
     <parent link="base_link" />
-    <child link="deimos_center" />
+    <child link="deimos_left_mount" />
   </joint>
 </robot>

Commit message: Added gazebo plugins, latest update from I3DR and removed pi property since xacro has it already

File: urdf/deimos.urdf.xacro (robot description, xacro)
@@ -2,7 +2,7 @@
 <!--
 Copyright (c) 2018, I3D Robotics Ltd.
+Edited: 2019, Marti Morta Garriga, Wood.
 -->
 <robot xmlns:xacro="http://ros.org/wiki/xacro">
-    <xacro:property name="M_PI" value="3.14159"/>
     <xacro:macro name="deimos_camera">
     <link name="cameraLeft_optical" />
@@ -13,8 +13,13 @@
         <visual>
             <origin xyz="0 0 0" rpy="0 0 0"/>
+            <!-- uncomment if using mesh as cad model is rotated -->
+            <!-- <origin xyz="0 0 0" rpy="${-pi/2} 0 ${-pi/2}"/> -->
             <geometry>
-                <box size="0.0324 0.101 0.038"/>
-                <!--mesh filename="package://deimos/urdf/deimos.stl" /-->
+                <box size="0.03242 0.10175 0.038"/>
+                <!-- <mesh filename="package://deimos/urdf/deimos.stl" /> -->
             </geometry>
+            <material name="Red">
+                <color rgba="0.9 0.1 0.1 1.0"/>
+            </material>
         </visual>
     </link>
@@ -28,20 +33,21 @@
         <parent link="deimos_left_mount"/>
         <child link="deimos_center"/>
-        <origin xyz="-0.13241 -${-0.017875+0.03} 0.025" rpy="0 0 0" />
+        <!-- <origin xyz="-0.13241 -${-0.017875+0.03} 0.025" rpy="0 0 0" comment="original" />  -->
+        <origin xyz="-0.013241 ${0.017875-0.03} 0.019" rpy="0 0 0" />
     </joint>
     <joint name="deimos_right_mount_joint" type="fixed">
         <parent link="deimos_left_mount"/>
         <child link="deimos_right_mount"/>
-        <origin xyz="0 0.03 0" rpy="0 0 0" />
+        <origin xyz="0 -0.03 0" rpy="0 0 0" />
     </joint>
     <joint name="deimos_right_camera_joint" type="fixed">
         <parent link="deimos_center"/>
         <child link="cameraRight"/>
-        <origin xyz="0 0.03 0" rpy="0 0 0" />
+        <origin xyz="0 -0.03 0" rpy="0 0 0" />
     </joint>
     <joint name="deimos_left_camera_joint" type="fixed">
         <parent link="deimos_center"/>
         <child link="cameraLeft"/>
-        <origin xyz="0 -0.03 0" rpy="0 0 0" />
+        <origin xyz="0 0.03 0" rpy="0 0 0" />
     </joint>
     <joint name="deimos_left_optical_joint" type="fixed">
@@ -49,5 +55,5 @@
         <child link="cameraLeft_optical"/>
 	<!-- Correct for the optical frame orientation -->
-        <origin xyz="0 0 0" rpy="${-M_PI/2} 0 ${-M_PI/2}" />
+        <origin xyz="0 0 0" rpy="${-pi/2} 0 ${-pi/2}" />
     </joint>
     <joint name="deimos_right_optical_joint" type="fixed">
@@ -55,5 +61,5 @@
         <child link="cameraRight_optical"/>
 	<!-- Correct for the optical frame orientation -->
-        <origin xyz="0 0 0" rpy="${-M_PI/2} 0 ${-M_PI/2}" />
+        <origin xyz="0 0 0" rpy="${-pi/2} 0 ${-pi/2}" />
     </joint>
     <joint name="deimos_depth_camera_joint" type="fixed">
@@ -64,8 +70,95 @@
     <!-- Correct for IMU orientation, Z -> X -->
     <joint name="imu_joint" type="fixed">
-    	<origin xyz="0 0.015 -0.002" rpy="0 ${M_PI/2} 0" />
+    	<origin xyz="0 0.015 -0.002" rpy="0 ${pi/2} 0" />
     	<parent link="deimos_center" />
     	<child link="imu_link" />
     </joint>
     </xacro:macro>
+     <gazebo reference="cameraLeft">
+            <sensor type="multicamera" name="stereo_camera">
+            <update_rate>0.5</update_rate> <!-- reality 60fps on USB3-->
+            <camera name="left">
+                <horizontal_fov>1.04</horizontal_fov>
+                <image>
+                    <width>752</width>
+                    <height>480</height>
+                    <format>L8</format>
+                </image>
+                <clip>
+                    <near>0.02</near>
+                    <far>300</far>
+                </clip>
+                <noise>
+                    <type>gaussian</type>
+                    <mean>0.0</mean>
+                    <stddev>0.007</stddev>
+                </noise>
+            </camera>
+            <camera name="right">
+                <pose>0 -0.07 0 0 0 0</pose>
+                <horizontal_fov>1.3962634</horizontal_fov>
+                <image>
+                    <width>752</width>
+                    <height>480</height>
+                    <format>L8</format>
+                </image>
+                <clip>
+                    <near>0.02</near>
+                    <far>300</far>
+                </clip>
+                <noise>
+                    <type>gaussian</type>
+                    <mean>0.0</mean>
+                    <stddev>0.007</stddev>
+                </noise>
+            </camera>
+            <plugin name="stereo_camera_controller" filename="libgazebo_ros_multicamera.so">
+                <alwaysOn>true</alwaysOn>
+                <updateRate>0.5</updateRate>
+                <cameraName>i3dr_deimos</cameraName>
+                <imageTopicName>image_raw</imageTopicName>
+                <cameraInfoTopicName>camera_info</cameraInfoTopicName>
+                <frameName>cameraLeft_optical</frameName>
+                <!--<rightFrameName>right_camera_optical_frame</rightFrameName>-->
+                <hackBaseline>0.07</hackBaseline>
+                <distortionK1>0.0</distortionK1>
+                <distortionK2>0.0</distortionK2>
+                <distortionK3>0.0</distortionK3>
+                <distortionT1>0.0</distortionT1>
+                <distortionT2>0.0</distortionT2>
+            </plugin>
+            </sensor>
+        </gazebo>
+        <gazebo reference="deimos_depth_camera">
+            <sensor type="depth" name="deimos_depth_camera">
+            <update_rate>0.5</update_rate>
+            <camera>
+                <horizontal_fov>${62.8 * pi/180.0}</horizontal_fov>
+                <image>
+                <format>R8G8B8</format>
+                <width>640</width>
+                <height>480</height>
+                </image>
+                <clip>
+                <near>0.05</near>
+                <far>12</far>
+                </clip>
+            </camera>
+            <plugin name="deimos_depth_camera_controller" filename="libgazebo_ros_openni_kinect.so">
+                <alwaysOn>true</alwaysOn>
+                <updateRate>0.5</updateRate>
+                <imageTopicName>i3dr_deimos_depth/image_raw</imageTopicName>
+                <cameraInfoTopicName>i3dr_deimos_depth/camera_info</cameraInfoTopicName>
+                <depthImageTopicName>i3dr_deimos_depth/depth/image_raw</depthImageTopicName>
+                <depthImageCameraInfoTopicName>i3dr_deimos_depth/depth/camera_info</depthImageCameraInfoTopicName>
+                <pointCloudTopicName>i3dr_deimos_depth/depth/points</pointCloudTopicName>
+                <frameName>cameraLeft_optical</frameName>
+                <distortion_k1>0.0</distortion_k1>
+                <distortion_k2>0.0</distortion_k2>
+                <distortion_k3>0.0</distortion_k3>
+                <distortion_t1>0.0</distortion_t1>
+                <distortion_t2>0.0</distortion_t2>
+            </plugin>
+            </sensor>
+    </gazebo>
 </robot>

Commit message: inital beta commit

File: urdf/deimos.urdf.xacro (robot description, xacro)
@@ -12,13 +12,10 @@
     <link name="deimos_center">
         <visual>
-            <origin xyz="0 0 0" rpy="0 0 0"/>
-            <!-- uncomment if using mesh as cad model is rotated -->
-            <!-- <origin xyz="0 0 0" rpy="${-pi/2} 0 ${-pi/2}"/> -->
+            <origin xyz="0 0 0" rpy="${pi/2} 0 ${pi/2}"/>
             <geometry>
-                <box size="0.03242 0.10175 0.038"/>
-                <!-- <mesh filename="package://deimos/urdf/deimos.stl" /> -->
+                <mesh filename="package://deimos/mesh/deimos.stl" />
             </geometry>
-            <material name="Red">
-                <color rgba="0.9 0.1 0.1 1.0"/>
+            <material name="Black">
+                <color rgba="0.1 0.1 0.1 1.0"/>
             </material>
         </visual>
@@ -33,5 +30,5 @@
         <parent link="deimos_left_mount"/>
         <child link="deimos_center"/>
-        <!-- <origin xyz="-0.13241 -${-0.017875+0.03} 0.025" rpy="0 0 0" comment="original" />  -->
+        <!--<origin xyz="0 0 0" rpy="0 0 0" />-->
         <origin xyz="-0.013241 ${0.017875-0.03} 0.019" rpy="0 0 0" />
     </joint>

Commit message: large merge

File: urdf/deimos.urdf.xacro (robot description, xacro)
@@ -5,30 +5,99 @@
 -->
 <robot xmlns:xacro="http://ros.org/wiki/xacro">
-    <xacro:macro name="deimos_camera">
-    <link name="cameraLeft_optical" />
-    <link name="cameraRight_optical" />
-    <link name="cameraLeft" />
-    <link name="cameraRight" />
-    <link name="deimos_center">
+    <xacro:macro name="deimos_camera" params="camera_name:=deimos en_mesh:=false imu_en:=false">
+    <xacro:property name="height" value="0.038"/>
+    <xacro:property name="width" value="0.10175"/>
+    <xacro:property name="length" value="0.03242"/>
+    <xacro:property name="mesh_file" value="package://i3dr_deimos/mesh/deimos.stl"/>
+    <xacro:property name="mesh_offset_xyz" value="-0.008 0.002 0"/>
+    <xacro:property name="mesh_offset_rpy" value="${pi/2} 0 ${pi/2}"/>
+    <xacro:property name="box_offset_xyz" value="0 0 0"/>
+    <xacro:property name="box_offset_rpy" value="0 0 0"/>
+    <link name="${camera_name}_cameraLeft_optical" />
+    <link name="${camera_name}_cameraRight_optical" />
+    <link name="${camera_name}_cameraLeft" />
+    <link name="${camera_name}_cameraRight" />
+    <link name="${camera_name}_depth_optical_frame" />
+    <link name="${camera_name}_base_link" />
+    <link name="${camera_name}_mount_point_1"/>
+    <link name="${camera_name}_mount_point_2"/>
+    <link name="${camera_name}_center">
         <visual>
-            <origin xyz="0 0 0" rpy="${pi/2} 0 ${pi/2}"/>
+            <xacro:if value="${(en_mesh == 'true')}">
+                <origin xyz="${mesh_offset_xyz}" rpy="${mesh_offset_rpy}"/>
+            </xacro:if>
+            <xacro:if value="${(en_mesh == 'false')}">
+                <origin xyz="${box_offset_xyz}" rpy="${box_offset_rpy}"/>
+            </xacro:if>
             <geometry>
-                <mesh filename="package://deimos/mesh/deimos.stl" />
+                <xacro:if value="${(en_mesh == 'true')}">
+                    <mesh filename="${mesh_file}"/>
+                </xacro:if>
+                <xacro:if value="${(en_mesh == 'false')}">
+                    <box size="${length} ${width} ${height}"/>
+                </xacro:if>
             </geometry>
-            <material name="Black">
-                <color rgba="0.1 0.1 0.1 1.0"/>
-            </material>
+            <xacro:if value="${(en_mesh == 'false')}">
+                <material name="${camera_name}_camera_colour">
+                    <color rgba="0.1 0.1 0.1 1.0"/>
+                </material>
+            </xacro:if>
         </visual>
     </link>
-    <link name="deimos_depth_camera" />
-    <link name="imu_link"/>
-    <!-- M4 trisert location -->
-    <link name="deimos_left_mount" />
-    <link name="deimos_right_mount" />
+    <joint name="${camera_name}_right_camera_joint" type="fixed">
+        <parent link="${camera_name}_center"/>
+        <child link="${camera_name}_cameraRight"/>
+        <origin xyz="0 ${-0.06/2}  0" rpy="0 0 0" />
+    </joint>
+    <joint name="${camera_name}_left_camera_joint" type="fixed">
+        <parent link="${camera_name}_center"/>
+        <child link="${camera_name}_cameraLeft"/>
+        <origin xyz="0 ${0.06/2}  0" rpy="0 0 0" />
+    </joint>
+    <joint name="${camera_name}_left_optical_joint" type="fixed">
+        <parent link="${camera_name}_cameraLeft"/>
+        <child link="${camera_name}_cameraLeft_optical"/>
+        <!-- Correct for the optical frame orientation -->
+        <origin xyz="0 0 0" rpy="${-pi/2} 0 ${(-pi/2)}" />
+    </joint>
+    <joint name="${camera_name}_right_optical_joint" type="fixed">
+        <parent link="${camera_name}_cameraRight"/>
+        <child link="${camera_name}_cameraRight_optical"/>
+        <!-- Correct for the optical frame orientation -->
+        <origin xyz="0 0 0" rpy="${-pi/2} 0 ${(-pi/2)}" />
+    </joint>
+    <joint name="${camera_name}_depth_optical_joint" type="fixed">
+        <parent link="${camera_name}_cameraLeft"/>
+        <child link="${camera_name}_depth_optical_frame"/>
+        <origin xyz="0 0 0" rpy="${-pi/2} 0 ${(-pi/2)}" />
+    </joint>
+    <joint name="${camera_name}_mount_center_joint" type="fixed">
+        <parent link="${camera_name}_base_link"/>
+        <child link="${camera_name}_center"/>
+        <origin xyz="0 0 0" rpy="0 0 ${-pi/2}" />
+    </joint>
+    <joint name="${camera_name}_mount_point_1_joint" type="fixed">
+        <parent link="${camera_name}_base_link"/>
+        <child link="${camera_name}_mount_point_1"/>
+        <origin xyz="${(0.03/2)-0.002} -0.007 ${-0.038/2}" rpy="0 0 0" />
+    </joint>
+    <joint name="${camera_name}_mount_point_2_joint" type="fixed">
+        <parent link="${camera_name}_base_link"/>
+        <child link="${camera_name}_mount_point_2"/>
+        <origin xyz="${(-0.03/2)-0.002} -0.007 ${-0.038/2}" rpy="0 0 0" />
+    </joint>
+    <xacro:if value="${(imu_en == 'true')}">
+        <!-- Correct for IMU orientation, Z -> X -->
+        <joint name="${camera_name}_imu_joint" type="fixed">
+            <origin xyz="0 0 0" rpy="0 ${pi/2} 0" />
+            <parent link="${camera_name}_imu_link" />
+            <child link="${camera_name}_base_link" />
+        </joint>
+    </xacro:if>
     <!-- Deimos has a 60 mm baseline -->
+    <!--
     <joint name="deimos_left_mount_joint" type="fixed">
         <parent link="deimos_left_mount"/>
         <child link="deimos_center"/>
-        <!--<origin xyz="0 0 0" rpy="0 0 0" />-->
         <origin xyz="-0.013241 ${0.017875-0.03} 0.019" rpy="0 0 0" />
     </joint>
@@ -48,27 +117,5 @@
         <origin xyz="0 0.03 0" rpy="0 0 0" />
     </joint>
-    <joint name="deimos_left_optical_joint" type="fixed">
-        <parent link="cameraLeft"/>
-        <child link="cameraLeft_optical"/>
-	<!-- Correct for the optical frame orientation -->
-        <origin xyz="0 0 0" rpy="${-pi/2} 0 ${-pi/2}" />
-    </joint>
-    <joint name="deimos_right_optical_joint" type="fixed">
-        <parent link="cameraRight"/>
-        <child link="cameraRight_optical"/>
-	<!-- Correct for the optical frame orientation -->
-        <origin xyz="0 0 0" rpy="${-pi/2} 0 ${-pi/2}" />
-    </joint>
-    <joint name="deimos_depth_camera_joint" type="fixed">
-        <parent link="cameraLeft"/>
-        <child link="deimos_depth_camera"/>
-        <origin xyz="0 0 0" rpy="0 0 0" />
-    </joint>
-    <!-- Correct for IMU orientation, Z -> X -->
-    <joint name="imu_joint" type="fixed">
-    	<origin xyz="0 0.015 -0.002" rpy="0 ${pi/2} 0" />
-    	<parent link="deimos_center" />
-    	<child link="imu_link" />
-    </joint>
+    -->
     </xacro:macro>
      <gazebo reference="cameraLeft">

File: urdf/deimos_scene.urdf.xacro (robot description, xacro)
@@ -5,5 +5,14 @@
 <robot name="deimos"
     xmlns:xacro="http://ros.org/wiki/xacro">
-    <xacro:include filename="$(find deimos)/urdf/i3dr_stereo_camera.urdf.xacro" />
-    <xacro:i3dr_stereo_camera camera_name="deimos" baseline="0.06" toe_in="0" width="0.038" height="0.10175" length="0.03242" mount_offset_y="-0.015" image_width="752" image_height="480" image_format="MONO8" hfov="1.04" focus_near="0.3" r="0.1" g="0.1" b="0.1" />
+    <!--<link name="odom"/>-->
+<!--
+    <xacro:include filename="$(find i3dr_stereo_camera)/urdf/i3dr_stereo_camera.urdf.xacro" />
+    <xacro:i3dr_stereo_camera camera_name="deimos" baseline="0.06" toe_in_r="0" toe_in_l="0" model_offset_xyz="-0.014 0 0" model_offset_rpy="1.57 0 1.57" width="0.10175" height="0.038" length="0.03242" imu_en="false" load_mesh="true" mesh_file="package://i3dr_deimos/mesh/deimos.stl" mount_offset_y="-0.015" image_width="752" image_height="480" image_format="MONO8" hfov="1.04" focus_near="0.3" r="0.1" g="0.1" b="0.1"/>
+-->
+    <xacro:include filename="$(find i3dr_deimos)/urdf/deimos.urdf.xacro" />
+    <xacro:deimos_camera camera_name="deimos" en_mesh="true"/>
+    <!--<joint name="world_imu_joint" type="floating">
+        <parent link="deimos_imu_link"/>
+        <child link="odom"/>
+    </joint>-->
 </robot>

Commit message: added probe mount link to urdf

File: urdf/deimos.urdf.xacro (robot description, xacro)
@@ -22,4 +22,5 @@
     <link name="${camera_name}_mount_point_1"/>
     <link name="${camera_name}_mount_point_2"/>
+    <link name="${camera_name}_probe_mount"/>
     <link name="${camera_name}_center">
         <visual>
@@ -76,4 +77,9 @@
         <child link="${camera_name}_center"/>
         <origin xyz="0 0 0" rpy="0 0 ${-pi/2}" />
+    </joint>
+    <joint name="${camera_name}_probe_mount_joint" type="fixed">
+        <parent link="${camera_name}_base_link"/>
+        <child link="${camera_name}_probe_mount"/>
+        <origin xyz="${0} 0 ${0}" rpy="0 0 0" />
     </joint>
     <joint name="${camera_name}_mount_point_1_joint" type="fixed">
